Commit message: URDF changes done

File: src/fwomni/urdf/fwomni.xacro (robot description, xacro)
@@ -4,4 +4,6 @@
 <xacro:include filename="$(find fwomni)/urdf/fwomni.trans" />
 <xacro:include filename="$(find fwomni)/urdf/fwomni.gazebo" />
+<link name="base_footprint">
+</link>
 <link name="base_link">
   <inertial>
@@ -11,5 +13,5 @@
   </inertial>
   <visual>
-    <origin xyz="0 0 0" rpy="0 0 0"/>
+    <origin xyz="0 0 0.005" rpy="0 0 0"/>
     <geometry>
       <mesh filename="package://fwomni/meshes/base_link.stl" scale="0.001 0.001 0.001"/>
@@ -18,5 +20,5 @@
   </visual>
   <collision>
-    <origin xyz="0 0 0" rpy="0 0 0"/>
+    <origin xyz="0 0 0.005" rpy="0 0 0"/>
     <geometry>
       <mesh filename="package://fwomni/meshes/base_link.stl" scale="0.001 0.001 0.001"/>
@@ -51,5 +53,5 @@
   </inertial>
   <visual>
-    <origin xyz="0.085328 -0.085328 0.005" rpy="0 0 0.785398"/>
+    <origin xyz="0 0 0" rpy="0 0 -1.5708"/>
     <geometry>
       <mesh filename="package://fwomni/meshes/wheel.stl" scale="0.001 0.001 0.001"/>
@@ -58,5 +60,5 @@
   </visual>
   <collision>
-    <origin xyz="0.085328 -0.085328 0.005" rpy="0 0 0.785398"/>
+    <origin xyz="0 0 0" rpy="0 0 -1.5708"/>
     <geometry>
       <mesh filename="package://fwomni/meshes/wheel.stl" scale="0.001 0.001 0.001"/>
@@ -71,5 +73,5 @@
   </inertial>
   <visual>
-    <origin xyz="0 0 0" rpy="0 0 0"/>
+    <origin xyz="0 0 0" rpy="0 0 -1.5708"/>
     <geometry>
       <mesh filename="package://fwomni/meshes/wheel.stl" scale="0.001 0.001 0.001"/>
@@ -78,5 +80,5 @@
   </visual>
   <collision>
-    <origin xyz="0 0 0" rpy="0 0 0"/>
+    <origin xyz="0 0 0" rpy="0 0 -1.5708"/>
     <geometry>
       <mesh filename="package://fwomni/meshes/wheel.stl" scale="0.001 0.001 0.001"/>
@@ -91,5 +93,5 @@
   </inertial>
   <visual>
-    <origin xyz="0 0 0" rpy="0 0 0"/>
+    <origin xyz="0 0 0" rpy="0 0 -1.5708"/>
     <geometry>
       <mesh filename="package://fwomni/meshes/wheel.stl" scale="0.001 0.001 0.001"/>
@@ -98,5 +100,5 @@
   </visual>
   <collision>
-    <origin xyz="0 0 0" rpy="0 0 0"/>
+    <origin xyz="0 0 0" rpy="0 0 -1.5708"/>
     <geometry>
       <mesh filename="package://fwomni/meshes/wheel.stl" scale="0.001 0.001 0.001"/>
@@ -111,5 +113,5 @@
   </inertial>
   <visual>
-    <origin xyz="0 0 0" rpy="0 0 0"/>
+    <origin xyz="0 0 0" rpy="0 0 -1.5708"/>
     <geometry>
       <mesh filename="package://fwomni/meshes/wheel.stl" scale="0.001 0.001 0.001"/>
@@ -118,5 +120,5 @@
   </visual>
   <collision>
-    <origin xyz="0 0 0" rpy="0 0 0"/>
+    <origin xyz="0 0 0" rpy="0 0 -1.5708"/>
     <geometry>
       <mesh filename="package://fwomni/meshes/wheel.stl" scale="0.001 0.001 0.001"/>
@@ -125,10 +127,15 @@
 </link>
 <joint name="Rigid1" type="fixed">
-  <origin xyz="0.065 0.0 0.025" rpy="0 0 0"/>
+  <origin xyz="0 0 0" rpy="0 0 0"/>
+  <parent link="base_footprint"/>
+  <child link="base_link"/>
+</joint>
+<joint name="Rigid2" type="fixed">
+  <origin xyz="0.065 0.0 0.03" rpy="0 0 0"/>
   <parent link="base_link"/>
   <child link="rplidar"/>
 </joint>
 <joint name="Cont1" type="continuous">
-  <origin xyz="0.085328 -0.085328 0.005" rpy="0 0 0.785398"/>
+  <origin xyz="0.085328 -0.085328 0.01" rpy="0 0 0.785398"/>
   <parent link="base_link"/>
   <child link="front_right"/>
@@ -136,5 +143,5 @@
 </joint>
 <joint name="Cont2" type="continuous">
-  <origin xyz="0.085328 0.085328 0.005" rpy="0 0 -0.785398"/>
+  <origin xyz="0.085328 0.085328 0.01" rpy="0 0 2.35619"/>
   <parent link="base_link"/>
   <child link="front_left"/>
@@ -142,5 +149,5 @@
 </joint>
 <joint name="Cont3" type="continuous">
-  <origin xyz="-0.085328 0.085328 0.005" rpy="0 0 0.785398"/>
+  <origin xyz="-0.085328 0.085328 0.01" rpy="0 0 -2.35619"/>
   <parent link="base_link"/>
   <child link="rear_left"/>
@@ -148,5 +155,5 @@
 </joint>
 <joint name="Cont4" type="continuous">
-  <origin xyz="-0.085328 -0.085328 0.005" rpy="0 0 -0.785398"/>
+  <origin xyz="-0.085328 -0.085328 0.01" rpy="0 0 -0.785398"/>
   <parent link="base_link"/>
   <child link="rear_right"/>

Commit message: RPLidar setup

File: src/fwomni/urdf/fwomni.xacro (robot description, xacro)
@@ -132,5 +132,5 @@
 </joint>
 <joint name="Rigid2" type="fixed">
-  <origin xyz="0.065 0.0 0.03" rpy="0 0 0"/>
+  <origin xyz="0.065 0.0 0.07" rpy="0 0 0"/>
   <parent link="base_link"/>
   <child link="rplidar"/>

Commit message: rotation achieved but not as expected

File: src/fwomni/urdf/fwomni.xacro (robot description, xacro)
@@ -9,5 +9,5 @@
   <inertial>
     <origin xyz="0.0014510929492462577 -1.1820705140781097e-17 0.00527905633638948" rpy="0 0 0"/>
-    <mass value="3.019927036453307"/>
+    <mass value="32.019927036453307"/>
     <inertia ixx="0.009026" iyy="0.009305" izz="0.018259" ixy="-0.0" iyz="-0.0" ixz="-5.4e-05"/>
   </inertial>
